Commit message: fixed go1 parameters with the most recent one from https://github.com/unitreerobotics/unitree_ros/blob/master/robots/go1_description/urdf/go1.urdf

File: quadruped_spring/go1_description/urdf/go1.urdf (robot description, URDF)
Before this commit: robot go1_description, 22 links, 21 joints
Links:
- link FL_calf: mass 0.158015 -> 0.131
- link FL_hip: mass 0.510299 -> 0.591
- link FL_thigh: mass 0.898919 -> 0.92
- link FR_calf: mass 0.158015 -> 0.131
- link FR_hip: mass 0.510299 -> 0.591
- link FR_thigh: mass 0.898919 -> 0.92
- link RL_calf: mass 0.158015 -> 0.131; geometry collision box size=0.213 0.016 0.016; visual mesh filename=package://go1_description/meshes/calf.stl scale=1 1 1
- link RL_hip: mass 0.510299 -> 0.591
- link RL_thigh: mass 0.898919 -> 0.92
- link RR_calf: mass 0.158015 -> 0.131
- link RR_hip: mass 0.510299 -> 0.591
- link RR_thigh: mass 0.898919 -> 0.92
- link trunk: mass 4.8 -> 5.204
Joints:
- joint FL_calf_joint: limit lower=-2.69653369433 upper=-0.916297857297 effort=33.5 velocity=21 -> lower=-2.72271363311 upper=-0.837758040957 effort=35.55 velocity=30.1
- joint FL_hip_joint: limit lower=-0.802851455917 upper=0.802851455917 effort=33.5 velocity=21 -> lower=-1.0471975512 upper=1.0471975512 effort=23.7 velocity=30.1
- joint FL_thigh_joint: limit lower=-1.0471975512 upper=4.18879020479 effort=33.5 velocity=21 -> lower=-0.663225115758 upper=2.96705972839 effort=23.7 velocity=30.1
- joint FR_calf_joint: limit lower=-2.69653369433 upper=-0.916297857297 effort=33.5 velocity=21 -> lower=-2.72271363311 upper=-0.837758040957 effort=35.55 velocity=30.1
- joint FR_hip_joint: limit lower=-0.802851455917 upper=0.802851455917 effort=33.5 velocity=21 -> lower=-1.0471975512 upper=1.0471975512 effort=23.7 velocity=30.1
- joint FR_thigh_joint: limit lower=-1.0471975512 upper=4.18879020479 effort=33.5 velocity=21 -> lower=-0.663225115758 upper=2.96705972839 effort=23.7 velocity=30.1
- joint RL_calf_joint: limit lower=-2.69653369433 upper=-0.916297857297 effort=33.5 velocity=21 -> lower=-2.72271363311 upper=-0.837758040957 effort=35.55 velocity=30.1
- joint RL_hip_joint: limit lower=-0.802851455917 upper=0.802851455917 effort=33.5 velocity=21 -> lower=-1.0471975512 upper=1.0471975512 effort=23.7 velocity=30.1
- joint RL_thigh_joint: limit lower=-1.0471975512 upper=4.18879020479 effort=33.5 velocity=21 -> lower=-0.663225115758 upper=2.96705972839 effort=23.7 velocity=30.1
- joint RR_calf_joint: limit lower=-2.69653369433 upper=-0.916297857297 effort=33.5 velocity=21 -> lower=-2.72271363311 upper=-0.837758040957 effort=35.55 velocity=30.1
- joint RR_hip_joint: limit lower=-0.802851455917 upper=0.802851455917 effort=33.5 velocity=21 -> lower=-1.0471975512 upper=1.0471975512 effort=23.7 velocity=30.1
- joint RR_thigh_joint: limit lower=-1.0471975512 upper=4.18879020479 effort=33.5 velocity=21 -> lower=-0.663225115758 upper=2.96705972839 effort=23.7 velocity=30.1

Commit message: modified the go1.urdf in according to unitree/pybullet/../a1.urdf

File: quadruped_spring/go1_description/urdf/go1.urdf (robot description, URDF)
Before this commit: robot go1_description, 22 links, 21 joints
Links:
- removed link FL_thigh_shoulder
- removed link FR_thigh_shoulder
- removed link RL_thigh_shoulder
- removed link RR_thigh_shoulder
- added link base, mass 0.00001; visual box size=0.001 0.001 0.001
- link FL_calf: geometry collision box size=0.213 0.016 0.016; visual mesh filename=package://go1_description/meshes/calf.obj scale=1 1 1
- link FL_hip: geometry collision cylinder length=0.04 radius=0.046; visual mesh filename=package://go1_description/meshes/hip.obj scale=1 1 1
- link FL_thigh: geometry collision box size=0.213 0.0245 0.034; visual mesh filename=package://go1_description/meshes/thigh.obj scale=1 1 1
- link FR_calf: geometry collision box size=0.213 0.016 0.016; visual mesh filename=package://go1_description/meshes/calf.obj scale=1 1 1
- link FR_hip: geometry collision cylinder length=0.04 radius=0.046; visual mesh filename=package://go1_description/meshes/hip.obj scale=1 1 1
- link FR_thigh: geometry collision box size=0.213 0.0245 0.034; visual mesh filename=package://go1_description/meshes/thigh_mirror.obj scale=1 1 1
- link RL_calf: geometry collision box size=0.213 0.016 0.016; visual mesh filename=package://go1_description/meshes/calf.obj scale=1 1 1
- link RL_hip: geometry collision cylinder length=0.04 radius=0.046; visual mesh filename=package://go1_description/meshes/hip.obj scale=1 1 1
- link RL_thigh: geometry collision box size=0.213 0.0245 0.034; visual mesh filename=package://go1_description/meshes/thigh.obj scale=1 1 1
- link RR_calf: geometry collision box size=0.213 0.016 0.016; visual mesh filename=package://go1_description/meshes/calf.obj scale=1 1 1
- link RR_hip: geometry collision cylinder length=0.04 radius=0.046; visual mesh filename=package://go1_description/meshes/hip.obj scale=1 1 1
- link RR_thigh: geometry collision box size=0.213 0.0245 0.034; visual mesh filename=package://go1_description/meshes/thigh_mirror.obj scale=1 1 1
Joints:
- removed joint FL_hip_fixed
- removed joint FR_hip_fixed
- removed joint RL_hip_fixed
- removed joint RR_hip_fixed
- added joint floating_base: type fixed, parent base, child trunk, origin xyz=0 0 0 rpy=0 0 0
